File: Xperimental_Trinket_Pro_small_parts_power_breakout.sch (EAGLE design)
At the start: 42 parts, among them J1 None, J2 None, SW1 None, U1 None, U2 None, U2A None, U2B None, Y1 16 MHz

Commit message: Better part parameter parsing
Fixed curvature of wires

Support for diodes

Multiple part database support

Standardized attributes

fixed tests

code for building GENERIC, RESOLVED, and UNRESOLVED devicesets automatically



git-svn-id: svn+ssh://bbfs-01.calit2.net/grw/Gordon/svn/trunk/Gadgets/Tools/CircuitsByCode@20112 2cf53259-273a-af40-bda6-69d31023b8ec
Parts:
- D1, D1A, D2, D2A, D2B, D5: value None -> <0.500V; DIST1 DigiKey -> (none); DIST1PN CRS08QMCT-ND -> (none); MFR Toshiba -> (none); MPN CRS08(TE85L,Q,M) -> (none); VFWD 0.25V -> (none)
- D3, D4: value None -> 3.6; DIST1 DigiKey -> (none); DIST1PN MM3Z3V6T1GOSCT-ND -> (none); MFR ON Semiconductor -> (none); MPN MM3Z3V6T1G -> (none); VZENER 3.6V -> (none)
- R2A: value 305K -> 305K+/-2%
- R2B: value 170K -> 170K+/-3%

Commit message: Resonator support.  Better tests and Makefiles
git-svn-id: svn+ssh://bbfs-01.calit2.net/grw/Gordon/svn/trunk/Gadgets/Tools/CircuitsByCode@20124 2cf53259-273a-af40-bda6-69d31023b8ec
Parts:
- Y1: DIST1 DigiKey -> (none); DIST1PN 490-1198-1-ND -> (none); MFR Murata -> (none); MPN CSTCE16M0V53-R0 -> (none); STBL 0.3% -> (none); TOL 0.5% -> (none)

Commit message: Cleaner error reporting.
Improved sanity checks.

Support for Device field in part databases

Removed terrible bug that was causing exponential slowdown over time by doubling the number of wires in the file every time it was loaded.  
Dramatic improvements in performance!

Fixed arduino schematic to only use GENERIC Components for things we can actually resolve.

Updated Base.lbr to support our new device model.





git-svn-id: svn+ssh://bbfs-01.calit2.net/grw/Gordon/svn/trunk/Gadgets/Tools/CircuitsByCode@20209 2cf53259-273a-af40-bda6-69d31023b8ec
Parts:
- C1, C1A, C1B, C2, C2A, C3, C4, C5: device NVSL:GENERIC-CAPACITOR-NP_2012-0805_CERAMIC -> NVSL:GENERIC-CAPACITOR-NP_
- D1, D1A, D2, D2A, D2B, D5: device NVSL:GENERIC-DIODE-SCHOTTKY_SOD323 -> NVSL:GENERIC-DIODE-SCHOTTKY_
- D3, D4: device NVSL:GENERIC-DIODE-ZENER_SOD323 -> NVSL:GENERIC-DIODE-ZENER_
- FTDI: device NVSL:GENERIC-SIP-6_2.54-SPACE-VERTICAL -> NVSL:SIP-6_2.54-SPACE-VERTICAL
- JP1: device NVSL:GENERIC-USB-5PIN-CONN_USB-MINIB-MTH-POSTS -> NVSL:USB-5PIN-CONN_USB-MINIB-MTH-POSTS
- JP3, JP4: device NVSL:GENERIC-SIP-12_2.54-SPACE-VERTICAL -> NVSL:SIP-12_2.54-SPACE-VERTICAL
- JP5: device NVSL:GENERIC-SIP-2_2.54-SPACE-VERTICAL -> NVSL:SIP-2_2.54-SPACE-VERTICAL
- LED1, LED2: device NVSL:GENERIC-DIODE-LED_2012-0805 -> NVSL:GENERIC-DIODE-LED_
- R1, R1A, R2A, R2B, R2C, R3, R4, R5, R6, R7, R8: device NVSL:GENERIC-RESISTOR_2012-0805_CERAMIC -> NVSL:GENERIC-RESISTOR_
- SW1: device NVSL:GENERIC-PUSHBUTTON-SHIELD-GND_CK_KMR211GLSR-TACTILE -> NVSL:PUSHBUTTON-SHIELD-GND_CK_KMR211GLSR-TACTILE
- U2, U2A, U2B: device NVSL:GENERIC-ADJUSTABLE-VOLTAGE-REGULATOR_SOIC8 -> NVSL:ADJUSTABLE-VOLTAGE-REGULATOR_SOIC8
- Y1: device NVSL:GENERIC-RESONATOR_V53-R0 -> NVSL:GENERIC-RESONATOR_
