File: Xperimental_Trinket_Pro_small_parts_power_breakout.sch (EAGLE design)
At the start: 42 parts, among them J1 None, J2 None, SW1 None, U1 None, U2 None, U2A None, U2B None, Y1 16 MHz

Commit message: More cleanup.  Split picker libraries into 'design' library and 'build' library.
git-svn-id: svn+ssh://bbfs-01.calit2.net/grw/Gordon/svn/trunk/Gadgets/Tools/CircuitsByCode@20258 2cf53259-273a-af40-bda6-69d31023b8ec
Parts:
- C1, C1A, C1B, C2, C2A, C3, C4, C5: device NVSL:GENERIC-CAPACITOR-NP_ -> PickerDesign:GENERIC-CAPACITOR-NP_
- D1, D1A, D2, D2A, D2B, D5: device NVSL:GENERIC-DIODE-SCHOTTKY_ -> PickerDesign:GENERIC-DIODE-SCHOTTKY_
- D3, D4: device NVSL:GENERIC-DIODE-ZENER_ -> PickerDesign:GENERIC-DIODE-ZENER_
- LED1, LED2: device NVSL:GENERIC-DIODE-LED_ -> PickerDesign:GENERIC-DIODE-LED_
- R1, R1A, R2A, R2B, R2C, R3, R4, R5, R6, R7, R8: device NVSL:GENERIC-RESISTOR_ -> PickerDesign:GENERIC-RESISTOR_
- Y1: device NVSL:GENERIC-RESONATOR_ -> PickerDesign:GENERIC-RESONATOR_

Commit message: More error handling.  The parser now correctly all of chris' tests files.  For the test files that match the eagle DTD, the output appears to match the input.  The match may not be perfect, but the input and output contain the same number and kind of tags and attributes.
git-svn-id: svn+ssh://bbfs-01.calit2.net/grw/Gordon/svn/trunk/Gadgets/Tools/CircuitsByCode@20342 2cf53259-273a-af40-bda6-69d31023b8ec
Parts:
- removed C1, C1A, C1B, C3: 3.3uF, PickerDesign:GENERIC-CAPACITOR-NP_
- removed C2, C2A: 100pF, PickerDesign:GENERIC-CAPACITOR-NP_
- removed C4, C5: 0.1uF, PickerDesign:GENERIC-CAPACITOR-NP_
- removed D1, D1A, D2, D2A, D2B, D5: <0.500V, PickerDesign:GENERIC-DIODE-SCHOTTKY_
- removed D3, D4: 3.6, PickerDesign:GENERIC-DIODE-ZENER_
- removed FTDI: None, NVSL:SIP-6_2.54-SPACE-VERTICAL
- removed J1, J2: None, NVSL:GENERIC-BATTERY-CONN-RECEPTACLEPH-SMD-2MM
- removed JP1: None, NVSL:USB-5PIN-CONN_USB-MINIB-MTH-POSTS
- removed JP3, JP4: None, NVSL:SIP-12_2.54-SPACE-VERTICAL
- removed JP5: None, NVSL:SIP-2_2.54-SPACE-VERTICAL
- removed LED1: Red, PickerDesign:GENERIC-DIODE-LED_
- removed LED2: Green, PickerDesign:GENERIC-DIODE-LED_
- removed R1, R1A: 100K, PickerDesign:GENERIC-RESISTOR_
- removed R2A: 305K+/-2%, PickerDesign:GENERIC-RESISTOR_
- removed R2B: 170K+/-3%, PickerDesign:GENERIC-RESISTOR_
- removed R2C: 143K, PickerDesign:GENERIC-RESISTOR_
- removed R3, R6: 470, PickerDesign:GENERIC-RESISTOR_
- removed R4, R5: 68, PickerDesign:GENERIC-RESISTOR_
- removed R7: 1.5K, PickerDesign:GENERIC-RESISTOR_
- removed R8: 10K, PickerDesign:GENERIC-RESISTOR_
- removed SW1: None, NVSL:PUSHBUTTON-SHIELD-GND_CK_KMR211GLSR-TACTILE
- removed U1: None, NVSL:ATMEGA328-NO-THERMAL_32TQFP
- removed U2, U2A, U2B: None, NVSL:ADJUSTABLE-VOLTAGE-REGULATOR_SOIC8
- removed Y1: 16 MHz, PickerDesign:GENERIC-RESONATOR_
Connections:
- removed net A0: JP3.7, U1.PC0(ADC0)
- removed net A1: JP3.8, U1.PC1(ADC1)
- removed net A2: JP3.9, U1.PC2(ADC2)
- removed net A3: JP3.10, U1.PC3(ADC3)
- removed net A4: JP3.11, U1.PC4(ADC4/SDA)
- removed net A5: JP3.12, U1.PC5(ADC5/SCL)
- removed net A6: JP5.1, U1.ADC6
- removed net A7: JP5.2, U1.ADC7
- removed net AREF: C5.1, JP3.6, U1.AREF
- removed net D+: D3.A, JP1.D+, R4.2
- removed net D-: D4.A, JP1.D-, R5.2, R7.1
- removed net D10: JP3.2, U1.PB2(SS/OC1B)
- removed net D11: JP3.3, U1.PB3(MOSI/OC2)
- removed net D12: JP3.4, U1.PB4(MISO)
- removed net D13: JP3.5, R6.1, U1.PB5(SCK)
- removed net D2: R4.1, U1.PD2(INT0)
- removed net D3: JP4.9, U1.PD3(INT1)
- removed net D4: JP4.8, U1.PD4(XCK/T0)
- removed net D5: JP4.7, U1.PD5(T1)
- removed net D6: JP4.6, U1.PD6(AIN0)
- removed net D7: R5.1, U1.PD7(AIN1)
- removed net D8: JP4.5, U1.PB0(ICP)
- removed net D9: JP3.1, U1.PB1(OC1A)
- removed net DTR/RTS: C4.2, FTDI.6
- removed net GND: C1.2, C1A.2, C1B.2, C3.2, C5.2, D3.C, D4.C, FTDI.1, FTDI.2, J1.2, J2.2, JP1.GND, JP4.2, LED1.C, LED2.C, R1.1, R1A.1, SW1.1, SW1.4, SW1.5, U1.GND, U1.GND@1, U1.GND@2, U2.GND, U2A.GND, U2B.GND, Y1.GND
- removed net N$2: LED1.A, R6.2
- removed net N$4: U1.PB7(XTAL2/TOSC2), Y1.OSC2
- removed net N$5: U1.PB6(XTAL1/TOSC1), Y1.OSC1
- removed net N$6: LED2.A, R3.1
- removed net RST: C4.1, JP4.12, R8.2, SW1.2, SW1.3, U1.PC6(/RESET)
- removed net RXD: FTDI.4, JP4.11, U1.PD0(RXD)
- removed net TXD: FTDI.5, JP4.10, U1.PD1(TXD)
- removed net VBAT: D1.A, D1A.A, D5.A, J1.1, J2.1, JP4.1
- removed net VBUS: D2.A, D2A.A, D2B.A, FTDI.3, JP1.VBUS, JP4.3
- removed net VCC: C2.1, C2A.1, C3.1, D2B.C, D5.C, JP4.4, R2A.2, R2B.2, R2C.2, R3.2, R7.2, R8.1, U1.AVCC, U1.VCC@1, U1.VCC@2, U2.OUT, U2A.OUT, U2B.OUT, U2B.SENSE
- removed net VFB: C2.2, C2A.2, R1.2, R1A.2, R2A.1, R2B.1, R2C.1, U2.FEEDB, U2A.FEEDB, U2B.FEEDB, U2B.VTAB
- removed net VIN: C1.1, C1A.1, C1B.1, D1.C, D1A.C, D2.C, D2A.C, U2.INPUT, U2A.INPUT, U2B.INPUT
Other:
- note removed: "(from 6-29V battery)"
- note removed: "(from USB)"
- note removed: "(power to the ATtiny)"
- note removed: "3.3V VCC!"
- note removed: "3V VCC!"
- note removed: "5V VCC !"
- note removed: "Adafruit Trinket 3.3/5V Modifed by UCSD"
- note removed: "Adafruit design modifed by SRD, at UCSD, CSE, NVSL Lab for educational use. Covered by Creative Commons Copyright via Adafruit."
- note removed: "Add this sheet 3 and pick a sheet 4, 5 etc. if you want to regulate USB or a battery voltage down to >= 1.24V CPU voltage."
- note removed: "Add this sheet if you wish to use USB 5V, unregulated and without a battery option."
- note removed: "Fixed 5V does not require R1 and R2 nor C2."
- note removed: "Insert Sheet 4 or 5 (resistor) for desired V."
- note removed: "Many load options here: This is a Universal Trinket that covers all power/load options. There will be separate break out sheets for variations on the power supplies etc. U2 Regulator is optional. Can use USB 5V PWR alone. Regulator VCC out controlled by R2. Regulator VIN can be VCC+0.5V to 29V. 3.6 to 6 VIN for 3 to 5 VCC recommended. D1, D2 and J2 only needed if Battery used. D5 protects USB if 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"
- note removed: "Note: Case grounded"
- note removed: "Note: NO Thermal"
- note removed: "SRD 9/14"
- note removed: "Selectively load R2 to adjust VCC, if used. ~305K 1% for 5V USB power ~170K 1% for 3.3V operation ~143K 1% for 3.0V etc. ** vout=~1.235 x (1+R2/100K) http://www.micrel.com/_PDF/mic2950.pdf 29V Max input on VBAT. Can use 220 Ohm on LEDs when running at 3.3V with plenty of power. The Schottky on VBAT is to protect USB in case battery is >5V and USB is plugged in by mistake. ** Note: When operating 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"
- note removed: "Substitute 174K 1% close enough - see BOM"
- note removed: "Substitute 309K 1% close enough - see BOM"
- note removed: "This 'Pro' design uses larger 0805 sizes and 1.27mm lead pitch whlere possible. Look elsewhere for a mostly 0603 & .635 mm based design. The processor package is the best available for hand soldering."
- note removed: "This 3V option may cause problems. See sheet 1 notes."
- note removed: "To design a Trinket, take this entire schematic, delete the sheets you do not need, switch to board, do the layout, and it "should just work." Be sure to error check to ensure you got it all."
- note removed: "Use one or more power supply pages that follow."
- note removed: "Use this sheet if you will operate ONLY at 5V from USB unregulated or ONLY at 5V regulated from battery."
- note removed: "Use this sheet instead of sheet 3 and pick a sheet 4 or 5 if you want to regulate USB down to >= 1.24V CPU voltage WITHOUT a battery option."
- note removed: "[ see http://adafruit.com/produts/1501 ]"
- note removed: "~ .25V forward drop each."
- note removed: "~ .25V forward drop."
