File: Xperimental_Trinket_Pro_small_parts_power_breakout.sch (EAGLE design)
At the start: 0 parts

Commit message: asciitree for library generation.  Moved tests for Koala and Swoop to python unittest.
git-svn-id: svn+ssh://bbfs-01.calit2.net/grw/Gordon/svn/trunk/Gadgets/Tools/CircuitsByCode@20442 2cf53259-273a-af40-bda6-69d31023b8ec
Parts:
- added C1, C1A, C1B, C3: 3.3uF, KoalaDesign:GENERIC-CAPACITOR-NP_
- added C2, C2A: 100pF, KoalaDesign:GENERIC-CAPACITOR-NP_
- added C4, C5: 0.1uF, KoalaDesign:GENERIC-CAPACITOR-NP_
- added D1, D1A, D2, D2A, D2B, D5: <0.500V, KoalaDesign:GENERIC-DIODE-SCHOTTKY_
- added D3, D4: 3.6, KoalaDesign:GENERIC-DIODE-ZENER_
- added FTDI: SIP-6_2.54-SPACE-VERTICAL, NVSL:SIP-6_2.54-SPACE-VERTICAL
- added J1, J2: GENERIC-BATTERY-CONN-RECEPTACLEPH-SMD-2MM, NVSL:GENERIC-BATTERY-CONN-RECEPTACLEPH-SMD-2MM
- added JP1: USB-5PIN-CONN_USB-MINIB-MTH-POSTS, NVSL:USB-5PIN-CONN_USB-MINIB-MTH-POSTS
- added JP3, JP4: SIP-12_2.54-SPACE-VERTICAL, NVSL:SIP-12_2.54-SPACE-VERTICAL
- added JP5: SIP-2_2.54-SPACE-VERTICAL, NVSL:SIP-2_2.54-SPACE-VERTICAL
- added LED1: Red, KoalaDesign:GENERIC-DIODE-LED_
- added LED2: Green, KoalaDesign:GENERIC-DIODE-LED_
- added R1, R1A: 100K, KoalaDesign:GENERIC-RESISTOR_
- added R2A: 305K+/-2%, KoalaDesign:GENERIC-RESISTOR_
- added R2B: 170K+/-3%, KoalaDesign:GENERIC-RESISTOR_
- added R2C: 143K, KoalaDesign:GENERIC-RESISTOR_
- added R3, R6: 470, KoalaDesign:GENERIC-RESISTOR_
- added R4, R5: 68, KoalaDesign:GENERIC-RESISTOR_
- added R7: 1.5K, KoalaDesign:GENERIC-RESISTOR_
- added R8: 10K, KoalaDesign:GENERIC-RESISTOR_
- added SW1: PUSHBUTTON-SHIELD-GND_CK_KMR211GLSR-TACTILE, NVSL:PUSHBUTTON-SHIELD-GND_CK_KMR211GLSR-TACTILE
- added U1: ATMEGA328-NO-THERMAL_32TQFP, NVSL:ATMEGA328-NO-THERMAL_32TQFP
- added U2, U2A, U2B: ADJUSTABLE-VOLTAGE-REGULATOR_SOIC8, NVSL:ADJUSTABLE-VOLTAGE-REGULATOR_SOIC8
- added Y1: 16 MHz, KoalaDesign:GENERIC-RESONATOR_
Connections:
- new net A0: JP3.7, U1.PC0(ADC0)
- new net A1: JP3.8, U1.PC1(ADC1)
- new net A2: JP3.9, U1.PC2(ADC2)
- new net A3: JP3.10, U1.PC3(ADC3)
- new net A4: JP3.11, U1.PC4(ADC4/SDA)
- new net A5: JP3.12, U1.PC5(ADC5/SCL)
- new net A6: JP5.1, U1.ADC6
- new net A7: JP5.2, U1.ADC7
- new net AREF: C5.1, JP3.6, U1.AREF
- new net D+: D3.A, JP1.D+, R4.2
- new net D-: D4.A, JP1.D-, R5.2, R7.1
- new net D10: JP3.2, U1.PB2(SS/OC1B)
- new net D11: JP3.3, U1.PB3(MOSI/OC2)
- new net D12: JP3.4, U1.PB4(MISO)
- new net D13: JP3.5, R6.1, U1.PB5(SCK)
- new net D2: R4.1, U1.PD2(INT0)
- new net D3: JP4.9, U1.PD3(INT1)
- new net D4: JP4.8, U1.PD4(XCK/T0)
- new net D5: JP4.7, U1.PD5(T1)
- new net D6: JP4.6, U1.PD6(AIN0)
- new net D7: R5.1, U1.PD7(AIN1)
- new net D8: JP4.5, U1.PB0(ICP)
- new net D9: JP3.1, U1.PB1(OC1A)
- new net DTR/RTS: C4.2, FTDI.6
- new net GND: C1.2, C1A.2, C1B.2, C3.2, C5.2, D3.C, D4.C, FTDI.1, FTDI.2, J1.2, J2.2, JP1.GND, JP4.2, LED1.C, LED2.C, R1.1, R1A.1, SW1.1, SW1.4, SW1.5, U1.GND, U1.GND@1, U1.GND@2, U2.GND, U2A.GND, U2B.GND, Y1.GND
- new net N$2: LED1.A, R6.2
- new net N$4: U1.PB7(XTAL2/TOSC2), Y1.OSC2
- new net N$5: U1.PB6(XTAL1/TOSC1), Y1.OSC1
- new net N$6: LED2.A, R3.1
- new net RST: C4.1, JP4.12, R8.2, SW1.2, SW1.3, U1.PC6(/RESET)
- new net RXD: FTDI.4, JP4.11, U1.PD0(RXD)
- new net TXD: FTDI.5, JP4.10, U1.PD1(TXD)
- new net VBAT: D1.A, D1A.A, D5.A, J1.1, J2.1, JP4.1
- new net VBUS: D2.A, D2A.A, D2B.A, FTDI.3, JP1.VBUS, JP4.3
- new net VCC: C2.1, C2A.1, C3.1, D2B.C, D5.C, JP4.4, R2A.2, R2B.2, R2C.2, R3.2, R7.2, R8.1, U1.AVCC, U1.VCC@1, U1.VCC@2, U2.OUT, U2A.OUT, U2B.OUT, U2B.SENSE
- new net VFB: C2.2, C2A.2, R1.2, R1A.2, R2A.1, R2B.1, R2C.1, U2.FEEDB, U2A.FEEDB, U2B.FEEDB, U2B.VTAB
- new net VIN: C1.1, C1A.1, C1B.1, D1.C, D1A.C, D2.C, D2A.C, U2.INPUT, U2A.INPUT, U2B.INPUT
Other:
- note added: "(from 6-29V battery)"
- note added: "(from USB)"
- note added: "(power to the ATtiny)"
- note added: "3.3V VCC!"
- note added: "3V VCC!"
- note added: "5V VCC !"
- note added: "Adafruit Trinket 3.3/5V Modifed by UCSD"
- note added: "Adafruit design modifed by SRD, at UCSD, CSE, NVSL Lab for educational use. Covered by Creative Commons Copyright via Adafruit."
- note added: "Add this sheet 3 and pick a sheet 4, 5 etc. if you want to regulate USB or a battery voltage down to >= 1.24V CPU voltage."
- note added: "Add this sheet if you wish to use USB 5V, unregulated and without a battery option."
- note added: "Fixed 5V does not require R1 and R2 nor C2."
- note added: "Insert Sheet 4 or 5 (resistor) for desired V."
- note added: "Many load options here: This is a Universal Trinket that covers all power/load options. There will be separate break out sheets for variations on the power supplies etc. U2 Regulator is optional. Can use USB 5V PWR alone. Regulator VCC out controlled by R2. Regulator VIN can be VCC+0.5V to 29V. 3.6 to 6 VIN for 3 to 5 VCC recommended. D1, D2 and J2 only needed if Battery used. D5 protects USB if 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"
- note added: "Note: Case grounded"
- note added: "Note: NO Thermal"
- note added: "SRD 9/14"
- note added: "Selectively load R2 to adjust VCC, if used. ~305K 1% for 5V USB power ~170K 1% for 3.3V operation ~143K 1% for 3.0V etc. ** vout=~1.235 x (1+R2/100K) http://www.micrel.com/_PDF/mic2950.pdf 29V Max input on VBAT. Can use 220 Ohm on LEDs when running at 3.3V with plenty of power. The Schottky on VBAT is to protect USB in case battery is >5V and USB is plugged in by mistake. ** Note: When operating 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"
- note added: "Substitute 174K 1% close enough - see BOM"
- note added: "Substitute 309K 1% close enough - see BOM"
- note added: "This 'Pro' design uses larger 0805 sizes and 1.27mm lead pitch whlere possible. Look elsewhere for a mostly 0603 & .635 mm based design. The processor package is the best available for hand soldering."
- note added: "This 3V option may cause problems. See sheet 1 notes."
- note added: "To design a Trinket, take this entire schematic, delete the sheets you do not need, switch to board, do the layout, and it "should just work." Be sure to error check to ensure you got it all."
- note added: "Use one or more power supply pages that follow."
- note added: "Use this sheet if you will operate ONLY at 5V from USB unregulated or ONLY at 5V regulated from battery."
- note added: "Use this sheet instead of sheet 3 and pick a sheet 4 or 5 if you want to regulate USB down to >= 1.24V CPU voltage WITHOUT a battery option."
- note added: "[ see http://adafruit.com/produts/1501 ]"
- note added: "~ .25V forward drop each."
- note added: "~ .25V forward drop."
