File: test2.sch (EAGLE design)
At the start: 4 parts

Commit message: More cleanup.  Split picker libraries into 'design' library and 'build' library.
git-svn-id: svn+ssh://bbfs-01.calit2.net/grw/Gordon/svn/trunk/Gadgets/Tools/CircuitsByCode@20258 2cf53259-273a-af40-bda6-69d31023b8ec
Parts:
- R1_3, R2_3, R3_3: device NVSL:GENERIC-RESISTOR_ -> PickerDesign:GENERIC-RESISTOR_

Commit message: Lots of documentation.  Code cleanup.  Got rid perl-generated intermeidate attribute file.  Fix for lists of attributes in <element>.  Some test boards and schematics.
git-svn-id: svn+ssh://bbfs-01.calit2.net/grw/Gordon/svn/trunk/Gadgets/Tools/CircuitsByCode@20352 2cf53259-273a-af40-bda6-69d31023b8ec
Parts:
- LED1_3: value None -> RGBLED_CA-5MM
Changed lines of the file:
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@@
       <parts>
         <part name="R1_3" library="PickerDesign" deviceset="GENERIC-RESISTOR_" device="" technology="" value="90 +/- 10%"/>
-        <part name="LED1_3" library="Components" deviceset="RGBLED_CA" device="-5MM" technology="" value="None">
+        <part name="LED1_3" library="Components" deviceset="RGBLED_CA" device="-5MM" technology="" value="">
           <attribute name="LUMENS" value=""/>
         </part>
