File: test/inputs/Trinket_Pro_default_SMD_parts_power_breakout.koala.sch (EAGLE design)
At the start: 42 parts, among them J1 None, J2 None, SW1 None, U1 None, U2 None, U2A None, U2B None, Y1 16 MHz

Commit message: fixed error handling
git-svn-id: svn+ssh://bbfs-01.calit2.net/grw/Gordon/svn/trunk/Gadgets/Tools/CircuitsByCode@21783 2cf53259-273a-af40-bda6-69d31023b8ec
Parts:
- FTDI: value None -> SIP-6_2.54-SPACE-VERTICAL
- J1, J2: value None -> BATTERY-CONN-RECEPTACLEPH-SMD-2MM
- JP1: value None -> USB-5PIN-CONN_USB-MINIB-MTH-POSTS
- JP3, JP4: value None -> SIP-12_2.54-SPACE-VERTICAL
- JP5: value None -> SIP-2_2.54-SPACE-VERTICAL
- SW1: value None -> PUSHBUTTON-SHIELD-GND_CK_KMR211GLSR-TACTILE
- U1: value None -> ATMEGA328-NO-THERMAL_32TQFP
- U2, U2A, U2B: value None -> ADJUSTABLE-VOLTAGE-REGULATOR_SOIC8
